File: PNPs/Toyota 4EFE/Fuel_Ignition.kicad_sch (KiCad schematic)
At the start: 49 parts, among them U1 VNLD5090, U2 IXDN602, U3 VNLD5090, U4 IXDN602

Commit message: Board layout done
Parts:
- removed C26: 0.1uF, Capacitor_SMD:C_0805_2012Metric, symbol Device:C
- removed C27: 1uF, Capacitor_SMD:C_0805_2012Metric, symbol Device:C
- removed D10, D4, D8, D9: LED, LED_SMD:LED_0805_2012Metric, symbol Device:LED
- removed D12, D6: D, Diode_SMD:D_SOD-323, symbol Device:D
- removed R10, R24, R25, R26: 2.4k, Resistor_SMD:R_0805_2012Metric, symbol Device:R
- removed R16, R19, R2, R20: 100k, Resistor_SMD:R_0805_2012Metric, symbol Device:R
- removed R18, R21, R22, R6: 1k, Resistor_SMD:R_0805_2012Metric, symbol Device:R
- removed R27, R28: 10R, Resistor_SMD:R_1206_3216Metric, symbol Device:R
- removed U4: IXDN602, Package_SO:SOIC-8_3.9x4.9mm_P1.27mm, symbol v0.4.4c-rescue:TC4424A-IC_Automotive
Connections:
- net INJ-3-OUT: no longer names the net of U3.6 (DRAIN2)
- net INJ-4-OUT: no longer names the net of U1.6 (DRAIN2)
Other:
- note removed: "Ignition Driver 2"
