File: PNPs/Toyota 4EFE/toyota 4efe.kicad_sch (KiCad schematic)
At the start: 1 part

Commit message: Added annotations etc.
Parts:
- XA1: footprint Shields:Arduino_Mega2560_Shield_IO_Only -> Library:Uno Shield
Changed lines of the file:
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@@
 			)
 		)
-		(property "Footprint" "Shields:Arduino_Mega2560_Shield_IO_Only"
+		(property "Footprint" "Library:Uno Shield"
 			(at 171.45 16.51 0)
 			(effects

Commit message: Board layout done
Parts:
- XA1: footprint Library:Uno Shield -> Shields:Arduino_Mega2560_Shield_IO_Only
Changed lines of the file:
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@@
 			)
 		)
-		(property "Footprint" "Library:Uno Shield"
+		(property "Footprint" "Shields:Arduino_Mega2560_Shield_IO_Only"
 			(at 171.45 16.51 0)
 			(effects
