File: PNPs/Toyota 4EFE/toyota 4efe.kicad_sch (KiCad schematic)
At the start: 1 part

Commit message: Added Mega shield, slight adjustments to traces
Parts:
- XA1: footprint Library:Uno Shield -> Library:Arduino_Mega2560_R3_Shield
Changed lines of the file:
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@@
 			)
 		)
-		(property "Footprint" "Library:Uno Shield"
+		(property "Footprint" "Library:Arduino_Mega2560_R3_Shield"
 			(at 171.45 16.51 0)
 			(effects
