File: PNPs/Toyota 4EFE/inputs.kicad_sch (KiCad schematic)
At the start: 40 parts, among them IC3 Trig Cond Socket, U5 MPX4250, U6 SP720

Commit message: Board layout done
Parts:
- removed JP2, JP3: VR-HALL, Connector_PinHeader_2.54mm:PinHeader_1x03_P2.54mm_Vertical, symbol Jumper:Jumper_3_Open
- removed JP4, JP5: PULL-UP, Connector_PinHeader_2.54mm:PinHeader_1x02_P2.54mm_Vertical, symbol Jumper:Jumper_2_Open
- removed R41, R42: 1k, Resistor_SMD:R_0805_2012Metric, symbol Device:R
- removed R43, R44: 220R, Resistor_SMD:R_0805_2012Metric, symbol Device:R
- U5: footprint Library:MPX5700ASX -> Misc:MPX4250
Connections:
- net CAM-IN: now also IC3.3 (Pin_3)
- net CRANK-IN: now also IC3.2 (Pin_2)

Commit message: Added annotations etc.
Parts:
- U5: footprint Misc:MPX4250 -> Library:MPX5700ASX
Changed lines of the file:
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@@
 			)
 		)
-		(property "Footprint" "Misc:MPX4250"
+		(property "Footprint" "Library:MPX5700ASX"
 			(at 49.53 48.26 0)
 			(effects
