File: PNPs/Toyota 4EFE/power.kicad_sch (KiCad schematic)
At the start: 12 parts, among them U8 LM2940S-5.0/NOPB

Commit message: Added Mega shield, slight adjustments to traces
Parts:
- C19: footprint Capacitor_SMD:C_0805_2012Metric_Pad1.15x1.40mm_HandSolder -> Capacitor_SMD:C_0805_2012Metric
Changed lines of the file:
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@@
 			)
 		)
-		(property "Footprint" "Capacitor_SMD:C_0805_2012Metric_Pad1.15x1.40mm_HandSolder"
+		(property "Footprint" "Capacitor_SMD:C_0805_2012Metric"
 			(at 140.97 126.6952 0)
 			(effects

Commit message: Board layout done
Parts:
- C19: footprint Capacitor_SMD:C_0805_2012Metric -> Capacitor_SMD:C_0805_2012Metric_Pad1.15x1.40mm_HandSolder
- S1: footprint Library:AYZ0202AGRLC -> Misc:AYZ0202AGRLC
Changed lines of the file:
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@@
 			)
 		)
-		(property "Footprint" "Library:AYZ0202AGRLC"
+		(property "Footprint" "Misc:AYZ0202AGRLC"
 			(at 176.53 125.73 0)
 			(effects
@@
 			)
 		)
-		(property "Footprint" "Capacitor_SMD:C_0805_2012Metric"
+		(property "Footprint" "Capacitor_SMD:C_0805_2012Metric_Pad1.15x1.40mm_HandSolder"
 			(at 140.97 126.6952 0)
 			(effects

Commit message: Added annotations etc.
Parts:
- S1: footprint Misc:AYZ0202AGRLC -> Library:AYZ0202AGRLC
Changed lines of the file:
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@@
 			)
 		)
-		(property "Footprint" "Misc:AYZ0202AGRLC"
+		(property "Footprint" "Library:AYZ0202AGRLC"
 			(at 176.53 125.73 0)
 			(effects
