File: PNPs/Toyota 4EFE/toyota 4efe.kicad_pcb (KiCad board)
At the start: 2 copper layers, 114 parts, among them IC3 Trig Cond Socket, J9 4E-FE OEM, Q2 SSM3K357R, Q3 SSM3K357R, U1 VNLD5090, U2 IXDN602, U3 VNLD5090, U4 IXDN602, U5 MPX4250, U6 SP720, U8 LM2940S-5.0/NOPB, U9 VNLD5090

Commit message: Board layout done
Parts:
- removed C26: 0.1uF, Capacitor_SMD:C_0805_2012Metric
- removed C27: 1uF, Capacitor_SMD:C_0805_2012Metric
- removed D10, D4, D8, D9: LED, LED_SMD:LED_0805_2012Metric
- removed D12, D6: D, Diode_SMD:D_SOD-323
- removed JP2, JP3: VR-HALL, Connector_PinHeader_2.54mm:PinHeader_1x03_P2.54mm_Vertical
- removed JP4, JP5: PULL-UP, Connector_PinHeader_2.54mm:PinHeader_1x02_P2.54mm_Vertical
- removed R10, R24, R25, R26: 2.4k, Resistor_SMD:R_0805_2012Metric
- removed R16, R19, R2, R20: 100k, Resistor_SMD:R_0805_2012Metric
- removed R18, R21, R22, R41, R42, R6: 1k, Resistor_SMD:R_0805_2012Metric
- removed R27, R28: 10R, Resistor_SMD:R_1206_3216Metric
- removed R43, R44: 220R, Resistor_SMD:R_0805_2012Metric
- removed U4: IXDN602, Package_SO:SOIC-8_3.9x4.9mm_P1.27mm
- added A1: Pololu_Breakout_DRV8825, Module:Pololu_Breakout-16_15.2x20.3mm, F.Cu at (125.4, 138.4)
- added D17: D, Diode_SMD:D_SOD-123F, F.Cu at (172.9, 121.4)
- added D18: D, Diode_SMD:D_SOD-123F, F.Cu at (172.8, 125.8)
- added R47: 1k, Resistor_SMD:R_0805_2012Metric, F.Cu at (158.6, 121.5)
- added R48: 1k, Resistor_SMD:R_0805_2012Metric, F.Cu at (158.6, 125.5)
- added R49: 100k, Resistor_SMD:R_0805_2012Metric, F.Cu at (154.8, 120.8)
- added R50: 100k, Resistor_SMD:R_0805_2012Metric, F.Cu at (154.8, 126.8)
- added U7: VNLD5090, Package_SO:SOIC-8_3.9x4.9mm_P1.27mm, F.Cu at (164.9, 123.5)
- moved C2 160.6 mm to (166.8, 53.4)
- moved D11 156.9 mm to (72.8, 52.7)
- moved C1 156.2 mm to (166.8, 56.8)
- moved C25 154.5 mm to (140.3, 49.6), turned to -90 degrees
- moved R34 153.5 mm to (167.6, 62.4), turned to 90 degrees
- moved JP11 153.3 mm to (162.9, 61.2), turned to 180 degrees
- moved C24 152.0 mm to (142.9, 49.7), turned to -90 degrees
- moved C20 151.1 mm to (60.0, 138.8), turned to 90 degrees
- moved C8 147.7 mm to (166.4, 67.3)
- moved JP1 146.8 mm to (136.9, 53.2), turned to 180 degrees
- moved U3 145.0 mm to (75.0, 48.6), turned to 180 degrees
- moved R23 143.9 mm to (76.7, 55.9), turned to 180 degrees
- moved C29 142.1 mm to (161.0, 73.8)
- moved U8 141.7 mm to (73.6, 146.4), turned to -90 degrees
- moved C18 141.1 mm to (73.7, 132.8), turned to -90 degrees
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Connections:
- IC3 pad 2: Net-(IC3-Pin_2) -> CRANK-IN
- IC3 pad 3: Net-(IC3-Pin_3) -> CAM-IN
- J9 pad 116: GND -> unconnected-(J9-Pad116)
- J9 pad 118: VCC -> VDD
- U1 pad 3: Net-(U1-IN2) -> unconnected-(U1-IN2-Pad3)
- U1 pad 6: INJ-4-OUT -> unconnected-(U1-DRAIN2-Pad6)
- U3 pad 3: Net-(U3-IN2) -> unconnected-(U3-IN2-Pad3)
- U3 pad 6: INJ-3-OUT -> unconnected-(U3-DRAIN2-Pad6)
Routing:
- net 12V-SW: track 0.00 -> 328.4 mm, vias 0 -> 5
- net MAP-EXT: track 0.00 -> 137.3 mm, vias 0 -> 2
- net TPS_Sensor: track 0.00 -> 113.8 mm, vias 0 -> 2
- net CLT_Sensor: track 0.00 -> 110.6 mm, vias 0 -> 2
- net MCU-D9: track 0.00 -> 104.3 mm
- net CRANK-IN: track 0.00 -> 102.4 mm
- net IAT_Sensor: track 0.00 -> 99.1 mm, vias 0 -> 2
- net MCU-D8: track 0.00 -> 94.4 mm
- net VDDA: track 0.00 -> 91.2 mm, vias 0 -> 2
- net VR1-: track 0.00 -> 90.5 mm
- net Vdrive: track 0.00 -> 84.3 mm, vias 0 -> 1
- net VDD: track 0.00 -> 82.9 mm, vias 0 -> 4
- net ADC-Clamp-2: track 0.00 -> 80.3 mm, vias 0 -> 3
- net O2_Sensor: track 0.00 -> 60.1 mm, vias 0 -> 2
- net ADC-Clamp-8: track 0.00 -> 57.5 mm
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- added copper zone on B.Cu, net GND
- added copper zone on F.Cu, net GND
- added copper zone on In1.Cu, net GND
- added copper zone on In2.Cu, net GND
- added copper zone on In2.Cu, net VDD
Other:
- copper layers 2 -> 4

Commit message: Added annotations etc.
Parts:
- removed Q3: SSM3K357R, Package_TO_SOT_SMD:SOT-23
- added J1: Conn_01x02, Connector_PinHeader_2.54mm:PinHeader_1x02_P2.54mm_Vertical, F.Cu at (177.4, 122.7)
- added J2: Conn_01x02, Connector_PinHeader_2.54mm:PinHeader_1x02_P2.54mm_Vertical, F.Cu at (177.6, 136.5)
- moved IC3 19.0 mm to (96.3, 128.0), turned to 0 degrees
- moved D16 7.57 mm to (166.0, 142.8), turned to 0 degrees
- moved D18 6.87 mm to (166.6, 128.6), turned to 0 degrees
- moved D19 6.18 mm to (166.7, 132.2), turned to 0 degrees
- moved D17 4.53 mm to (168.9, 119.4), turned to 0 degrees
- moved Q2 3.32 mm to (86.5, 75.7)
- moved C24 0.83 mm to (143.7, 49.7)
Routing:
- net CRANK-IN: track 102.4 -> 79.2 mm
- net VR1-: track 90.5 -> 72.8 mm
- net HC-2-OUT: track 3.48 -> 16.8 mm
- net HC-1-OUT: track 4.82 -> 16.8 mm
- net IDLE-OUT: track 4.00 -> 14.7 mm
- net BOOST-OUT: track 4.29 -> 14.3 mm
- net MCU-D45: track 7.82 -> 0.00 mm
- net 12V-SW: track 328.4 -> 321.4 mm
- net ADC-Clamp-9: track 55.1 -> 48.4 mm
- net MCU-D47: track 10.3 -> 7.16 mm
- net ADC-Clamp-8: track 57.5 -> 54.7 mm
- net FAN-OUT: track 42.8 -> 41.4 mm
- net Vdrive: track 84.3 -> 85.1 mm
Other:
- board text added: "12V"
- board text added: "5V"
- board text added: "ALIGN"
- board text added: "BOOST OUT HC-1 OUT"
- board text added: "IDLE OUT HC-2 OUT"
- board text added: "IGN-1 OUT"
- board text added: "IGN-2 OUT"
- board text added: "IGNITION VOLTAGE"
- board text added: "INJ-1 OUT"
- board text added: "INJ-2 OUT"
- board text added: "Stepper Driver"
- board text added: "TOYOTA 4E-FE PnP SPEEDUINO COMPATIBLE ECU BOARD v0.1 Designed by Henrik Heininen"
- board text added: "Trigger Conditioner Socket"
